File: Hardware/Aktorbaustein_v2.5/Aktorbaustein.kicad_pcb (KiCad board)
At the start: 2 copper layers, 150 x 72 mm, 106 parts, among them IC1 FT231XS-U, J1 TB001-500-02BE, J10 TB003V-500-P02BE, J11 CON-SOCJ-2155, J2 TB001-500-02BE, J3 TB001-500-02BE, J4 TB001-500-02BE, J5 TB002-500-03BE, J6 TB002-500-03BE, J7 TB002-500-03BE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

Commit message: Soos
Parts:
- moved H3 3.10 mm to (41.1, 107.9)
- moved H1 3.10 mm to (41.1, 44.1)
Routing:
- net DTR: track 45.8 -> 44.5 mm, vias 1 -> 0
Other:
- board text removed: "K2"
- board text removed: "K3"
- board text removed: "K4"

Commit message: soos
Routing:
- net +3V3: track 388.2 -> 387.5 mm
Changed lines of the file:
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@@
   (layers
     (0 F.Cu signal)
-    (31 B.Cu signal hide)
+    (31 B.Cu signal)
     (32 B.Adhes user)
     (33 F.Adhes user)
@@
       (drillshape 0)
       (scaleselection 1)
-      (outputdirectory ""))
+      (outputdirectory "C:/Users/FT12L/Documents/KiCad/projekt5/actuator_module_v2/"))
   )
   (net 0 "")
@@
   (segment (start 92.684999 60.264999) (end 82.085001 60.264999) (width 0.25) (layer F.Cu) (net 10))
   (segment (start 82.085001 60.264999) (end 78.25 64.1) (width 0.25) (layer F.Cu) (net 10))
-  (via (at 99.05 70.85) (size 0.8) (drill 0.4) (layers F.Cu B.Cu) (net 10))
-  (segment (start 99.05 76.65) (end 99.05 70.85) (width 0.25) (layer F.Cu) (net 10))
   (segment (start 92 82.45) (end 93.25 82.45) (width 0.25) (layer F.Cu) (net 10))
-  (segment (start 93.25 82.45) (end 99.05 76.65) (width 0.25) (layer F.Cu) (net 10))
-  (via (at 99.1 68.8) (size 0.8) (drill 0.4) (layers F.Cu B.Cu) (net 10))
-  (segment (start 99.05 70.85) (end 99.05 68.85) (width 0.25) (layer B.Cu) (net 10))
-  (segment (start 99.05 68.85) (end 99.1 68.8) (width 0.25) (layer B.Cu) (net 10))
-  (segment (start 96.8 66.5) (end 95.7 66.5) (width 0.25) (layer F.Cu) (net 10))
-  (segment (start 99.1 68.8) (end 96.8 66.5) (width 0.25) (layer F.Cu) (net 10))
   (segment (start 67.6 104.8) (end 67.6 105.9) (width 0.25) (layer B.Cu) (net 10))
   (via (at 67.6 107.35) (size 0.8) (drill 0.4) (layers F.Cu B.Cu) (net 10))
@@
   (segment (start 172.3636 89.95001) (end 174.14999 89.95001) (width 0.25) (layer F.Cu) (net 10))
   (segment (start 174.14999 89.95001) (end 174.5 90.30002) (width 0.25) (layer F.Cu) (net 10))
+  (segment (start 92 80.75) (end 98.2 74.55) (width 0.25) (layer F.Cu) (net 10))
+  (segment (start 92 82.45) (end 92 80.75) (width 0.25) (layer F.Cu) (net 10))
+  (via (at 98.2 70.425) (size 0.8) (drill 0.4) (layers F.Cu B.Cu) (net 10))
+  (segment (start 98.2 74.55) (end 98.2 70.425) (width 0.25) (layer F.Cu) (net 10))
+  (via (at 98.2 68.7) (size 0.8) (drill 0.4) (layers F.Cu B.Cu) (net 10))
+  (segment (start 98.2 70.425) (end 98.2 68.7) (width 0.25) (layer B.Cu) (net 10))
+  (segment (start 96 66.5) (end 95.7 66.5) (width 0.25) (layer F.Cu) (net 10))
+  (segment (start 98.2 68.7) (end 96 66.5) (width 0.25) (layer F.Cu) (net 10))
   (segment (start 105.4 80.45) (end 105.4 71.5) (width 0.25) (layer F.Cu) (net 11))
   (segment (start 107.5 81.5) (end 106.45 81.5) (width 0.25) (layer F.Cu) (net 11))
