File: Hardware/Aktorbaustein_v2.5/Logik.sch (KiCad schematic (older format))
At the start: 39 parts, among them IC1 FT231XS-U, J10 TB003V-500-P02BE, J11 CON-SOCJ-2155, J9 Conn_01x06_Male, Q5 MMBT3904, Q6 MMBT3904, SW1 SKHHALA010, SW2 SKHHALA010, SW3 SKHHALA010, U2 ESP32-WROOM-32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

Commit message: zgzgzg
Parts:
- SW1: Vendor (none) -> 688-SKHHAL; vendor 688-SKHHAL -> (none)
Changed lines of the file:
@@
 F 3 "~" H 1850 3750 50  0001 C CNN
 F 4 "clear" V 1850 3800 50  0000 C CNN "comment"
-F 5 "688-SKHHAL" V 1850 3550 50  0001 C CNN "vendor"
+F 5 "688-SKHHAL" V 1850 3550 50  0001 C CNN "Vendor"
 	1    1850 3550
 	0    1    1    0
