File: Hardware/Aktorbaustein_v2.5/Schnittstellen.sch (KiCad schematic (older format))
At the start: 63 parts, among them J1 TB001-500-02BE, J2 TB001-500-02BE, J3 TB001-500-02BE, J4 TB001-500-02BE, J5 TB002-500-03BE, J6 TB002-500-03BE, J7 TB002-500-03BE, J8 TB002-500-03BE, K1 G5LE-1-VD DC24, K2 G5LE-1-VD DC24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

Commit message: zgzgzg
Parts:
- R21, R22: Vendor 660-RN73H1JTD4702F25 -> 755-KTR03EZPF3302
- R23, R25: Vendor 660-RN73H1JTD2002D25 -> 660-RN73H1JTD1203F25
- R24, R26: Vendor 660-RN73H1JTD2002D25 -> 755-KTR03EZPF1102
- R8: Vednor 71-CRCW0603100KFKEAC -> (none); Vendor (none) -> 71-CRCW0603100KFKEAC
Changed lines of the file:
@@
 F 2 "Resistor_SMD:R_0603_1608Metric_Pad1.05x0.95mm_HandSolder" V 9280 1150 50  0001 C CNN
 F 3 "~" H 9350 1150 50  0001 C CNN
-F 4 "660-RN73H1JTD2002D25" H 9350 1150 50  0001 C CNN "Vendor"
+F 4 "755-KTR03EZPF1102" H 9350 1150 50  0001 C CNN "Vendor"
 	1    9350 1150
 	1    0    0    -1
@@
 F 2 "Resistor_SMD:R_0603_1608Metric_Pad1.05x0.95mm_HandSolder" V 9030 1000 50  0001 C CNN
 F 3 "~" H 9100 1000 50  0001 C CNN
-F 4 "660-RN73H1JTD4702F25" V 9100 1000 50  0001 C CNN "Vendor"
+F 4 "755-KTR03EZPF3302" V 9100 1000 50  0001 C CNN "Vendor"
 	1    9100 1000
 	0    -1   -1   0
@@
 F 2 "Resistor_SMD:R_0603_1608Metric_Pad1.05x0.95mm_HandSolder" V 9330 2850 50  0001 C CNN
 F 3 "~" H 9400 2850 50  0001 C CNN
-F 4 "660-RN73H1JTD2002D25" H 9400 2850 50  0001 C CNN "Vendor"
+F 4 "755-KTR03EZPF1102" H 9400 2850 50  0001 C CNN "Vendor"
 	1    9400 2850
 	1    0    0    -1
@@
 F 2 "Resistor_SMD:R_0603_1608Metric_Pad1.05x0.95mm_HandSolder" V 9080 2700 50  0001 C CNN
 F 3 "~" H 9150 2700 50  0001 C CNN
-F 4 "660-RN73H1JTD4702F25" V 9150 2700 50  0001 C CNN "Vendor"
+F 4 "755-KTR03EZPF3302" V 9150 2700 50  0001 C CNN "Vendor"
 	1    9150 2700
 	0    -1   -1   0
@@
 F 2 "Resistor_SMD:R_0603_1608Metric_Pad1.05x0.95mm_HandSolder" V 1680 7300 50  0001 C CNN
 F 3 "~" H 1750 7300 50  0001 C CNN
-F 4 "71-CRCW0603100KFKEAC" H 1750 7300 50  0001 C CNN "Vednor"
+F 4 "71-CRCW0603100KFKEAC" H 1750 7300 50  0001 C CNN "Vendor"
 	1    1750 7300
 	1    0    0    -1
@@
 F 2 "Resistor_SMD:R_0603_1608Metric_Pad1.05x0.95mm_HandSolder" V 9280 850 50  0001 C CNN
 F 3 "~" H 9350 850 50  0001 C CNN
-F 4 "660-RN73H1JTD2002D25" H 9350 850 50  0001 C CNN "Vendor"
+F 4 "660-RN73H1JTD1203F25" H 9350 850 50  0001 C CNN "Vendor"
 	1    9350 850
 	1    0    0    -1
@@
 F 2 "Resistor_SMD:R_0603_1608Metric_Pad1.05x0.95mm_HandSolder" V 9330 2550 50  0001 C CNN
 F 3 "~" H 9400 2550 50  0001 C CNN
-F 4 "660-RN73H1JTD2002D25" H 9400 2550 50  0001 C CNN "Vendor"
+F 4 "660-RN73H1JTD1203F25" H 9400 2550 50  0001 C CNN "Vendor"
 	1    9400 2550
 	1    0    0    -1
