File: Hardware/Frontplatte_v1.6/Frontplatte.sch (KiCad schematic (older format))
At the start: 14 parts, among them J1 61000621121

Commit message: zgzgzg
Parts:
- D1, D2, D3, D4: value 156120RS75000 -> 156120GS75000; Vendor 710-156120RS75000 -> 710-156120GS75000
- J1: Vendor (none) -> 710-61000621121; mouser 710-61000621121 -> (none)
- R1, R2, R3, R4: value 100 -> 220; Vendor 660-RN73H1JT1000F100 -> 71-CRCW0603220RJNEBC
Changed lines of the file:
@@
 P 5300 2950
 F 0 "D1" H 5293 2695 50  0000 C CNN
-F 1 "156120RS75000" H 5293 2786 50  0000 C CNN
+F 1 "156120GS75000" H 5293 2786 50  0000 C CNN
 F 2 "reverse_LED:reverse_mounted_LED_hole_2.3mm" H 5300 2950 50  0001 C CNN
 F 3 "~" H 5300 2950 50  0001 C CNN
-F 4 "710-156120RS75000" H 5300 2950 50  0001 C CNN "Vendor"
+F 4 "710-156120GS75000" H 5300 2950 50  0001 C CNN "Vendor"
 	1    5300 2950
 	-1   0    0    1
@@
 P 5300 3400
 F 0 "D2" H 5293 3145 50  0000 C CNN
-F 1 "156120RS75000" H 5293 3236 50  0000 C CNN
+F 1 "156120GS75000" H 5293 3236 50  0000 C CNN
 F 2 "reverse_LED:reverse_mounted_LED_hole_2.3mm" H 5300 3400 50  0001 C CNN
 F 3 "~" H 5300 3400 50  0001 C CNN
-F 4 "710-156120RS75000" H 5300 3400 50  0001 C CNN "Vendor"
+F 4 "710-156120GS75000" H 5300 3400 50  0001 C CNN "Vendor"
 	1    5300 3400
 	-1   0    0    1
@@
 P 5300 3800
 F 0 "D3" H 5293 3545 50  0000 C CNN
-F 1 "156120RS75000" H 5293 3636 50  0000 C CNN
+F 1 "156120GS75000" H 5293 3636 50  0000 C CNN
 F 2 "reverse_LED:reverse_mounted_LED_hole_2.3mm" H 5300 3800 50  0001 C CNN
 F 3 "~" H 5300 3800 50  0001 C CNN
-F 4 "710-156120RS75000" H 5300 3800 50  0001 C CNN "Vendor"
+F 4 "710-156120GS75000" H 5300 3800 50  0001 C CNN "Vendor"
 	1    5300 3800
 	-1   0    0    1
@@
 P 5300 4200
 F 0 "D4" H 5293 3945 50  0000 C CNN
-F 1 "156120RS75000" H 5293 4036 50  0000 C CNN
+F 1 "156120GS75000" H 5293 4036 50  0000 C CNN
 F 2 "reverse_LED:reverse_mounted_LED_hole_2.3mm" H 5300 4200 50  0001 C CNN
 F 3 "~" H 5300 4200 50  0001 C CNN
-F 4 "710-156120RS75000" H 5300 4200 50  0001 C CNN "Vendor"
+F 4 "710-156120GS75000" H 5300 4200 50  0001 C CNN "Vendor"
 	1    5300 4200
 	-1   0    0    1
@@
 P 4850 2950
 F 0 "R1" V 4643 2950 50  0000 C CNN
-F 1 "100" V 4734 2950 50  0000 C CNN
+F 1 "220" V 4734 2950 50  0000 C CNN
 F 2 "Resistor_SMD:R_0603_1608Metric_Pad1.05x0.95mm_HandSolder" V 4780 2950 50  0001 C CNN
 F 3 "~" H 4850 2950 50  0001 C CNN
-F 4 "660-RN73H1JT1000F100" V 4850 2950 50  0001 C CNN "Vendor"
+F 4 "71-CRCW0603220RJNEBC" V 4850 2950 50  0001 C CNN "Vendor"
 	1    4850 2950
 	0    1    1    0
@@
 P 4850 3800
 F 0 "R3" V 4643 3800 50  0000 C CNN
-F 1 "100" V 4734 3800 50  0000 C CNN
+F 1 "220" V 4734 3800 50  0000 C CNN
 F 2 "Resistor_SMD:R_0603_1608Metric_Pad1.05x0.95mm_HandSolder" V 4780 3800 50  0001 C CNN
 F 3 "~" H 4850 3800 50  0001 C CNN
-F 4 "660-RN73H1JT1000F100" V 4850 3800 50  0001 C CNN "Vendor"
+F 4 "71-CRCW0603220RJNEBC" V 4850 3800 50  0001 C CNN "Vendor"
 	1    4850 3800
 	0    1    1    0
@@
 P 4850 3400
 F 0 "R2" V 4643 3400 50  0000 C CNN
-F 1 "100" V 4734 3400 50  0000 C CNN
+F 1 "220" V 4734 3400 50  0000 C CNN
 F 2 "Resistor_SMD:R_0603_1608Metric_Pad1.05x0.95mm_HandSolder" V 4780 3400 50  0001 C CNN
 F 3 "~" H 4850 3400 50  0001 C CNN
-F 4 "660-RN73H1JT1000F100" V 4850 3400 50  0001 C CNN "Vendor"
+F 4 "71-CRCW0603220RJNEBC" V 4850 3400 50  0001 C CNN "Vendor"
 	1    4850 3400
 	0    1    1    0
@@
 P 4850 4200
 F 0 "R4" V 4643 4200 50  0000 C CNN
-F 1 "100" V 4734 4200 50  0000 C CNN
+F 1 "220" V 4734 4200 50  0000 C CNN
 F 2 "Resistor_SMD:R_0603_1608Metric_Pad1.05x0.95mm_HandSolder" V 4780 4200 50  0001 C CNN
 F 3 "~" H 4850 4200 50  0001 C CNN
-F 4 "660-RN73H1JT1000F100" V 4850 4200 50  0001 C CNN "Vendor"
+F 4 "71-CRCW0603220RJNEBC" V 4850 4200 50  0001 C CNN "Vendor"
 	1    4850 4200
 	0    1    1    0
@@
 F 2 "Connector_PinHeader_2.54mm:PinHeader_2x06_P2.54mm_Vertical_SMD" H 8700 3200 50  0001 C CNN
 F 3 "~" H 8700 3200 50  0001 C CNN
-F 4 "710-61000621121" H 8700 3200 50  0001 C CNN "mouser"
+F 4 "710-61000621121" H 8700 3200 50  0001 C CNN "Vendor"
 	1    8700 3200
 	1    0    0    1
