File: Hardware/Sensorbaustein_v3.5/Sensorbaustein.sch (KiCad schematic (older format))
At the start: 37 parts, among them IC1 FT231XS-U, J1 Conn_01x02_Male, J2 Conn_01x02_Male, J3 Conn_02x06_Odd_Even, Q1 MMBT2222ALT1G, Q2 MMBT2222ALT1G, U1 ESP32-WROOM-32

Commit message: zgzgzg
Parts:
- C1: Vendor (none) -> 81-GRM188R60J106ME4J
- D2, D3, D4, D5, D6, D7, D8, D9: Vendor (none) -> 583-BAT54
- IC1: Vendor (none) -> 895-FT231XS-U
- J3: Vendor (none) -> 437-8038701210001101
- S1, S2, S3: Vendor (none) -> 688-SKTHAHE010
Changed lines of the file:
@@
 EESchema Schematic File Version 4
+LIBS:Sensorbaustein-cache
 EELAYER 30 0
 EELAYER END
@@
 F 10 "895-FT231XS-U" H 4400 2850 50  0001 L CNN "Mouser Part Number"
 F 11 "https://www.mouser.co.uk/ProductDetail/FTDI/FT231XS-U?qs=Gp1Yz1mis3WFP7tMtj2Z9g%3D%3D" H 4400 2750 50  0001 L CNN "Mouser Price/Stock"
+F 12 "895-FT231XS-U" H 3250 3550 50  0001 C CNN "Vendor"
 	1    3250 3550
 	1    0    0    -1
@@
 F 2 "Capacitor_SMD:C_0603_1608Metric_Pad1.05x0.95mm_HandSolder" H 1988 3950 50  0001 C CNN
 F 3 "~" H 1950 4100 50  0001 C CNN
+F 4 "81-GRM188R60J106ME4J" H 1950 4100 50  0001 C CNN "Vendor"
 	1    1950 4100
 	1    0    0    -1
@@
 F 2 "Diode_SMD:D_SOT-23_ANK" H 1000 1200 50  0001 C CNN
 F 3 "~" H 1000 1200 50  0001 C CNN
+F 4 "583-BAT54" V 1000 1200 50  0001 C CNN "Vendor"
 	1    1000 1200
 	0    1    1    0
@@
 F 2 "Diode_SMD:D_SOT-23_ANK" H 1000 900 50  0001 C CNN
 F 3 "~" H 1000 900 50  0001 C CNN
+F 4 "583-BAT54" V 1000 900 50  0001 C CNN "Vendor"
 	1    1000 900
 	0    1    1    0
@@
 F 2 "Diode_SMD:D_SOT-23_ANK" H 1000 2350 50  0001 C CNN
 F 3 "~" H 1000 2350 50  0001 C CNN
+F 4 "583-BAT54" V 1000 2350 50  0001 C CNN "Vendor"
 	1    1000 2350
 	0    1    1    0
@@
 F 2 "Diode_SMD:D_SOT-23_ANK" H 1000 2050 50  0001 C CNN
 F 3 "~" H 1000 2050 50  0001 C CNN
+F 4 "583-BAT54" V 1000 2050 50  0001 C CNN "Vendor"
 	1    1000 2050
 	0    1    1    0
@@
 F 2 "Connector_PinSocket_2.54mm:PinSocket_2x06_P2.54mm_Vertical" H 3600 1250 50  0001 C CNN
 F 3 "~" H 3600 1250 50  0001 C CNN
-F 4 "" H 3600 1250 50  0001 C CNN "mouser"
+F 4 "437-8038701210001101" H 3600 1250 50  0001 C CNN "Vendor"
 	1    3600 1250
 	-1   0    0    1
@@
 F 2 "Diode_SMD:D_SOT-23_ANK" H 1900 2350 50  0001 C CNN
 F 3 "~" H 1900 2350 50  0001 C CNN
+F 4 "583-BAT54" V 1900 2350 50  0001 C CNN "Vendor"
 	1    1900 2350
 	0    1    1    0
@@
 F 2 "Diode_SMD:D_SOT-23_ANK" H 1900 2050 50  0001 C CNN
 F 3 "~" H 1900 2050 50  0001 C CNN
+F 4 "583-BAT54" V 1900 2050 50  0001 C CNN "Vendor"
 	1    1900 2050
 	0    1    1    0
@@
 F 2 "Diode_SMD:D_SOT-23_ANK" H 1900 1200 50  0001 C CNN
 F 3 "~" H 1900 1200 50  0001 C CNN
+F 4 "583-BAT54" V 1900 1200 50  0001 C CNN "Vendor"
 	1    1900 1200
 	0    1    1    0
@@
 F 2 "Diode_SMD:D_SOT-23_ANK" H 1900 900 50  0001 C CNN
 F 3 "~" H 1900 900 50  0001 C CNN
+F 4 "583-BAT54" V 1900 900 50  0001 C CNN "Vendor"
 	1    1900 900
 	0    1    1    0
@@
 F 4 "1.8mm" H 8750 4450 50  0001 L BNN "Feld4"
 F 5 "Manufacturer recommendations" H 8750 4450 50  0001 L BNN "Feld5"
-F 6 "" H 8750 4450 50  0001 L BNN "Feld6"
+F 6 "688-SKTHAHE010" H 8750 4450 50  0001 L BNN "Vendor"
 	1    8750 4450
 	0    1    1    0
@@
 F 4 "1.8mm" H 9650 4450 50  0001 L BNN "Feld4"
 F 5 "Manufacturer recommendations" H 9650 4450 50  0001 L BNN "Feld5"
-F 6 "" H 9650 4450 50  0001 L BNN "Feld6"
+F 6 "688-SKTHAHE010" H 9650 4450 50  0001 L BNN "Vendor"
 	1    9650 4450
 	0    1    1    0
@@
 F 4 "1.8mm" H 10550 4450 50  0001 L BNN "Feld4"
 F 5 "Manufacturer recommendations" H 10550 4450 50  0001 L BNN "Feld5"
-F 6 "" H 10550 4450 50  0001 L BNN "Feld6"
+F 6 "688-SKTHAHE010" H 10550 4450 50  0001 L BNN "Vendor"
 	1    10550 4450
 	0    1    1    0
